File: Mitayi-Pico-RP2040.kicad_pcb (KiCad board)
At the start: 2 copper layers, 43.8 x 51 mm, 53 parts, among them J2 USB_C_Receptacle_USB2.0, Q1 NMOS, U1 W25Q128JVS, U2 MIC5219-3.3YM5, U3 RP2040, U4 DS18B20Z, U5 SHT31-DIS, U6 DS18B20Z, X1 12MHz Yangxing Tech X322512MS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

Commit message: Even more parts
Parts:
- SW_BOOT1, SW_RESET1: footprint 00_Project:TS-1187A-B-A-B -> 00_Project:SW_TS-1187A-B-A-B
- U5: footprint Sensor_Humidity:Sensirion_DFN-8-1EP_2.5x2.5mm_P0.5mm_EP1.1x1.7mm -> 00_Project:SON50P250X250X90-9T110X180N
- moved SW_BOOT1 8.90 mm to (119.1, 69.1)
- moved SW_RESET1 8.90 mm to (119.1, 78.8)
Other:
- board text added: "*"

Commit message: Cleanup
Parts:
- removed R1: DNP, Resistor_SMD:R_0402_1005Metric_Pad0.72x0.64mm_HandSolder
- U1: value W25Q128JVS -> W25Q128JVSIQ
Connections:
- Q1 pad 3: unconnected-(Q1-S-Pad3) -> GND
- R2 pad 2: /~{USB_BOOT} -> Net-(SW_BOOT1-A)
- SW_BOOT1 pad 1: /~{USB_BOOT} -> GND
- SW_BOOT1 pad 2: /~{USB_BOOT} -> GND
- SW_BOOT1 pad 3: GND -> Net-(SW_BOOT1-A)
- SW_BOOT1 pad 4: GND -> Net-(SW_BOOT1-A)
- U1 pad 1: unconnected-(U1-~{CS}-Pad1) -> /QSPI_SS
- U1 pad 2: unconnected-(U1-DO(IO1)-Pad2) -> /QSPI_SD1
- U1 pad 3: unconnected-(U1-IO2-Pad3) -> /QSPI_SD2
- U1 pad 4: unconnected-(U1-GND-Pad4) -> GND
- U1 pad 5: unconnected-(U1-DI(IO0)-Pad5) -> /QSPI_SD0
- U1 pad 6: unconnected-(U1-CLK-Pad6) -> /QSPI_SCLK
- U1 pad 7: unconnected-(U1-IO3-Pad7) -> /QSPI_SD3
- U1 pad 8: unconnected-(U1-VCC-Pad8) -> +3V3
Routing:
- net /QSPI_SD0: track 0.00 -> 16.4 mm
- net /QSPI_SD3: track 0.00 -> 14.4 mm, vias 0 -> 2
- net /QSPI_SCLK: track 0.00 -> 14.3 mm, vias 0 -> 2
- net Net-(SW_BOOT1-A): track 0.00 -> 14.3 mm
- net /~{USB_BOOT}: track 10.4 -> 0.00 mm
- net /QSPI_SD2: track 0.00 -> 8.01 mm
- net /QSPI_SD1: track 0.00 -> 7.69 mm
- net GND: track 9.44 -> 14.5 mm, vias 33 -> 32
- net /GPIO11: track 24.8 -> 22.1 mm
- net +3V3: track 139.6 -> 138.2 mm
- net /GPIO12: track 19.4 -> 18.7 mm
