File: Mitayi-Pico-RP2040.kicad_sch (KiCad schematic)
At the start: 53 parts, among them J2 USB_C_Receptacle_USB2.0, Q1 NMOS, U1 W25Q128JVS, U2 MIC5219-3.3YM5, U3 RP2040, U4 DS18B20Z, U5 SHT31-DIS, U6 DS18B20Z, X1 12MHz Yangxing Tech X322512MS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

Commit message: Even more parts
Parts:
- SW_BOOT1, SW_RESET1: footprint 00_Project:TS-1187A-B-A-B -> 00_Project:SW_TS-1187A-B-A-B
- U5: footprint Sensor_Humidity:Sensirion_DFN-8-1EP_2.5x2.5mm_P0.5mm_EP1.1x1.7mm -> 00_Project:SON50P250X250X90-9T110X180N
Changed lines of the file:
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@@
       (effects (font (size 1.27 1.27)) (justify left))
     )
-    (property "Footprint" "Sensor_Humidity:Sensirion_DFN-8-1EP_2.5x2.5mm_P0.5mm_EP1.1x1.7mm" (at 113.03 222.25 0)
+    (property "Footprint" "00_Project:SON50P250X250X90-9T110X180N" (at 113.03 222.25 0)
       (effects (font (size 1.27 1.27)) hide)
     )
@@
       (effects (font (size 0.8 0.8)))
     )
-    (property "Footprint" "00_Project:TS-1187A-B-A-B" (at 52.07 214.63 0)
+    (property "Footprint" "00_Project:SW_TS-1187A-B-A-B" (at 52.07 214.63 0)
       (effects (font (size 1.27 1.27)) hide)
     )
@@
       (effects (font (size 0.8 0.8)))
     )
-    (property "Footprint" "00_Project:TS-1187A-B-A-B" (at 46.99 171.45 0)
-      (effects (font (size 1.27 1.27)) hide)
-    )
+    (property "Footprint" "00_Project:SW_TS-1187A-B-A-B" (at 46.99 171.45 0)
+      (effects (font (size 1.27 1.27)) hide)
+    )

Commit message: Cleanup
Parts:
- removed R1: DNP, Resistor_SMD:R_0402_1005Metric_Pad0.72x0.64mm_HandSolder, symbol Device:R
- U1: value W25Q128JVS -> W25Q128JVSIQ; JCL (none) -> C97521
Connections:
- net +3V3: now also U1.8 (VCC)
- net GND: now also Q1.3 (S), SW_BOOT1.1, SW_BOOT1.2, U1.4 (GND); no longer SW_BOOT1.3 (K), SW_BOOT1.4 (A)
- net QSPI_SCLK: now also U1.6 (CLK)
- net QSPI_SD0: now also U1.5 (DI(IO0))
- net QSPI_SD1: now also U1.2 (DO(IO1))
- net QSPI_SD2: now also U1.3 (IO2)
- net QSPI_SD3: now also U1.7 (IO3)
- net QSPI_SS: now also U1.1 (~{CS})
- removed net ~{USB_BOOT}: R2.2, SW_BOOT1.1, SW_BOOT1.2
- new net: R2.2, SW_BOOT1.3 (K), SW_BOOT1.4 (A)
Other:
- note removed: "DEB_EN"
- note removed: "Not required by all Flash. -> Use 10K if needed."
- note removed: "There are JVS and FVS versions. -> JVS is faster."
- note removed: "User Button"
- moved on the sheet: C1, C13, C14, C15, C16, C17, C18, C19, C20, D1, D2, D3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
